File: hardware/v2-double-sided/kicad_pcb/esp32FC.kicad_sch (KiCad schematic)
At the start: 30 parts, among them J1 Conn_01x05_Pin, J10 Screw_Terminal_01x02, J11 Screw_Terminal_01x02, J12 Screw_Terminal_01x02, J2 Conn_01x04_Pin, J3 Conn_01x03_Pin, J4 Conn_01x03_Pin, J5 Conn_01x03_Pin, J6 Conn_01x03_Pin, J7 Screw_Terminal_01x02, J8 Screw_Terminal_01x02, J9 Screw_Terminal_01x02, Q1 2N3904, U1 esp32-wemos-d1-mini

Commit message: Added screw holes and export files
Other:
- title: (none) -> ESP32FC - PCB for X Quadcopter Drones
Changed lines of the file:
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@@
 	(generator_version "9.0")
 	(paper "A4")
+	(title_block
+		(title "ESP32FC - PCB for X Quadcopter Drones")
+		(date "2025-06-29")
+		(rev "v2.0")
+	)
 	(junction
 		(at 102.87 39.37)

Commit message: Modified connectors for serial connections, now used molex connectors
Parts:
- removed J1: Conn_01x05_Pin, Connector_PinHeader_2.54mm:PinHeader_1x05_P2.54mm_Vertical, symbol Connector:Conn_01x05_Pin
- added J1: Conn_01x06_Pin, Connector_Molex:Molex_KK-254_AE-6410-06A_1x06_P2.54mm_Vertical, symbol Connector:Conn_01x06_Pin
- J2: footprint Connector_PinHeader_2.54mm:PinHeader_1x04_P2.54mm_Vertical -> Connector_Molex:Molex_KK-254_AE-6410-04A_1x04_P2.54mm_Vertical
- renumbered C6 to C3, C7 to C4, C3 to C5, C4 to C6, C5 to C7, J7 to J12, J12 to J7, R3 to R2, R4 to R3, R5 to R4
Connections:
- net +3.3V: now also J1.4 (Pin_4)
- net +5V: now also J2.3 (Pin_3), J1.2 (Pin_2); no longer J2.2 (Pin_2)
- net GND: now also J2.4 (Pin_4), J1.3 (Pin_3); no longer J2.1 (Pin_1)
- net RX2: now also J2.2 (Pin_2); no longer J2.3 (Pin_3)
- net RX3: now also J1.6 (Pin_6)
- net TX2: now also J2.1 (Pin_1); no longer J2.4 (Pin_4)
- net TX3: now also J1.5 (Pin_5)
- no-connect marks 24 -> 25

Commit message: Added two additional outs, to connect two additional servos
Parts:
- added J7, J8: Conn_01x03_Pin, Connector_PinHeader_2.54mm:PinHeader_1x03_P2.54mm_Vertical, symbol Connector:Conn_01x03_Pin
- renumbered J8 to J10, J9 to J11, J10 to J12, J11 to J13, J12 to J14, J7 to J9, R2 to R1, R3 to R2, R1 to R3
Connections:
- net GND: now also J7.3 (Pin_3), J8.3 (Pin_3)
- net M1: now also J3.1 (Pin_1); no longer J6.1 (Pin_1)
- net M2: now also J4.1 (Pin_1); no longer J5.1 (Pin_1)
- net M3: now also J5.1 (Pin_1), U1.28 (IO_32); no longer J3.1 (Pin_1), U1.32 (IO_04)
- net M4: now also J6.1 (Pin_1); no longer J4.1 (Pin_1)
- net SERVO2: now reaches U1.34 (IO_00)
- net SERVO2: now also J8.1 (Pin_1)
- new net SERVO1: J7.1 (Pin_1), U1.32 (IO_04)
Other:
- moved on the sheet: BZ1, J1, J2, J3, J4, J5, J6, Q1, R3
